File: RocketLocator.kicad_sch (KiCad schematic)
At the start: 118 parts, among them J1 USB_C, J12 Battery / Switch, J2 Deploy Ch1 / Ch2, J3 Battery-, J4 Deploy Ch3 / Ch4, J7 U.FL-R-SMT(01), J8 Conn_ST_STDC14, Q1 2N7002KN, Q3 BSS84, Q4 PMXB43UNE, Q5 PMXB43UNE, Q6 PMXB43UNE, Q7 PMXB43UNE, U1 TPS22950YBHR, U11 PAM8904EGPR, U12 74HCS00, U13 DMP2021UFDF, U14 ISM6HG256XTR, U15 TPS22950YBHR, U16 MS5611-01BA, U17 MX25L6436F, U18 BQ25185DLHR, U2 SAM-M10Q-00B, U3 DRV5032DUDMRR, U4 CH340N, U5 STM32WL5MOCH6TR, U6 TPS22950YBHR, U7 RT9080-33GJ5, U8 TPS22950YBHR, U9 TPS22950YBHR

Commit message: Move C7 (BATTLVL filter) to 0402 X7R
C7 only filters the battery-sense divider node (max ~3.2 V), so the
out-of-stock 50 V C0G 1206 part is not needed. Swap it to the same
0.1uF 0402 X7R as the other decoupling caps (C1525):
- Schematic footprint Capacitor_SMD:C_0402_1005Metric
- PCB: 0402 placed vertically on B.Cu at (41.775, 30.16) on the
  existing BATTLVL node; GND pad picks up the B.Cu pour. Old GND stub
  removed, zones refilled. DRC: 0 errors, 0 unconnected, schematic
  parity clean.
- BOM: C7 merged into the 0.1uF row, its own row removed.

Co-Authored-By: Claude Opus 5.5 (1M context) <noreply@anthropic.com>
Claude-Session: https://claude.ai/code/session_01Qn4Fhe37cECFfk8PPTy8Kj
Parts:
- C7: footprint Capacitor_SMD:C_1206_3216Metric -> Capacitor_SMD:C_0402_1005Metric
Changed lines of the file:
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@@
 			)
 		)
-		(property "Footprint" "Capacitor_SMD:C_1206_3216Metric"
+		(property "Footprint" "Capacitor_SMD:C_0402_1005Metric"
 			(at 260.6548 109.22 0)
 			(hide yes)

Commit message: Add MMC5983MA magnetometer on I2C2
U19 MMC5983MA (JLCPCB C404329) joins the GPS I2C bus at 0x30 with
SPI_CS tied to VDDIO for I2C mode. C38 1uF on VDD, C39 0.1uF on VDDIO,
C37 10uF on CAP for the SET/RESET pulse. INT and SPI_SDO left unconnected.
Footprint is KiCad's stock Package_LGA:LGA-16_3x3mm_P0.5mm, which matches
the datasheet land pattern. New Custom:MMC5983MA symbol. BOM updated.

Co-Authored-By: Claude Opus 5.5 (1M context) <noreply@anthropic.com>
Claude-Session: https://claude.ai/code/session_01FYY8Uv6gBjRSv3QTZNtnYK
Parts:
- added C37: 10uF, Capacitor_SMD:C_0402_1005Metric, symbol Device:C
- added C38: 1uF, Capacitor_SMD:C_0402_1005Metric, symbol Device:C
- added C39: 0.1uF, Capacitor_SMD:C_0402_1005Metric, symbol Device:C
- added U19: MMC5983MA, Package_LGA:LGA-16_3x3mm_P0.5mm, symbol Custom:MMC5983MA
Connections:
- net $SCL: now also U19.1 (SCL/SPI_SCK)
- net $SDA: now also U19.16 (SDA/SPI_SDI)
- net +3V3: now also C38.1, C39.1, U19.13 (VDDIO), U19.2 (VDD), U19.4 (~{SPI_CS})
- net GND: now also C37.2, C38.2, C39.2, U19.11 (GND), U19.9 (GND)
- new net: C37.1, U19.10 (CAP)
- new net: U19.12 (NC), U19.14 (NC), U19.3 (NC), U19.6 (NC), U19.7 (NC), U19.8 (NC)
- no-connect marks 28 -> 30
Other:
- note added: "Magnetometer I2C 0x30"
