File: RocketLocator.kicad_sch (KiCad schematic)
At the start: 122 parts, among them J1 USB_C, J12 Battery / Switch, J2 Deploy Ch1 / Ch2, J3 Battery-, J4 Deploy Ch3 / Ch4, J7 U.FL-R-SMT(01), J8 Conn_ST_STDC14, Q1 2N7002KN, Q3 BSS84, Q4 PMXB43UNE, Q5 PMXB43UNE, Q6 PMXB43UNE, Q7 PMXB43UNE, U1 TPS22950YBHR, U11 PAM8904EGPR, U12 74HCS00, U13 DMP2021UFDF, U14 ISM6HG256XTR, U15 TPS22950YBHR, U16 MS5611-01BA, U17 MX25L6436F, U18 BQ25185DLHR, U19 MMC5983MA, U2 SAM-M10Q-00B, U3 DRV5032DUDMRR, U4 CH340N, U5 STM32WL5MOCH6TR, U6 TPS22950YBHR, U7 RT9080-33GJ5, U8 TPS22950YBHR, U9 TPS22950YBHR

Commit message: Drop C39 VDDIO bypass cap to match MMC5983MA datasheet
The datasheet application circuit has only 1uF on VDD (C38) and 10uF on
CAP (C37); VDD and VDDIO share +3V3 here, so C38 covers both.

Co-Authored-By: Claude Opus 5.5 (1M context) <noreply@anthropic.com>
Claude-Session: https://claude.ai/code/session_01FYY8Uv6gBjRSv3QTZNtnYK
Parts:
- removed C39: 0.1uF, Capacitor_SMD:C_0402_1005Metric, symbol Device:C
Changed lines of the file:
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@@
 	)
 	(junction
-		(at 81.28 243.84)
-		(diameter 0)
-		(color 0 0 0 0)
-	)
-	(junction
 		(at 172.72 209.55)
 		(diameter 0)
@@
 	)
 	(symbol
-		(lib_id "power:GND")
-		(at 81.28 251.46 0)
-		(unit 1)
-		(body_style 1)
-		(exclude_from_sim no)
-		(in_bom yes)
-		(on_board yes)
-		(in_pos_files yes)
-		(dnp no)
-		(property "Reference" "#GND0213"
-			(at 81.28 257.81 0)
-			(hide yes)
-			(show_name no)
-			(do_not_autoplace no)
-			(effects
-				(font
-					(size 1.27 1.27)
-				)
-			)
-		)
-		(property "Value" "GND"
-			(at 81.153 255.8542 0)
-			(show_name no)
-			(do_not_autoplace no)
-			(effects
-				(font
-					(size 1.27 1.27)
-				)
-			)
-		)
-		(property "Footprint" ""
-			(at 81.28 251.46 0)
-			(hide yes)
-			(show_name no)
-			(do_not_autoplace no)
-			(effects
-				(font
-					(size 1.27 1.27)
-				)
-			)
-		)
-		(property "Datasheet" ""
-			(at 81.28 251.46 0)
-			(hide yes)
-			(show_name no)
-			(do_not_autoplace no)
-			(effects
-				(font
-					(size 1.27 1.27)
-				)
-			)
-		)
-		(property "Description" ""
-			(at 81.28 251.46 0)
-			(hide yes)
-			(show_name no)
-			(do_not_autoplace no)
-			(effects
-				(font
-					(size 1.27 1.27)
-				)
-			)
-		)
-		(pin "1"
-		)
-		(instances
-			(project "RocketLocator"
-				(path "/e63e39d7-6ac0-4ffd-8aa3-1841a4541b55"
-					(reference "#GND0213")
-					(unit 1)
-				)
-			)
-		)
-	)
-	(symbol
 		(lib_id "Custom:74HC00")
 		(at 195.58 43.18 0)
@@
 					(unit 1)
 				)
-			)
-		)
-	)
-	(symbol
-		(lib_id "Device:C")
-		(at 81.28 247.65 0)
-		(unit 1)
-		(body_style 1)
-		(exclude_from_sim no)
-		(in_bom yes)
-		(on_board yes)
-		(in_pos_files yes)
-		(dnp no)
-		(property "Reference" "C39"
-			(at 83.82 246.38 0)
-			(show_name no)
-			(do_not_autoplace no)
-			(effects
-				(font
-					(size 1.27 1.27)
-				)
-				(justify left)
-			)
-		)
-		(property "Value" "0.1uF"
-			(at 83.82 248.92 0)
-			(show_name no)
-			(do_not_autoplace no)
-			(effects
-				(font
-					(size 1.27 1.27)
-				)
-				(justify left)
-			)
-		)
-		(property "Footprint" "Capacitor_SMD:C_0402_1005Metric"
-			(at 80.3148 251.46 0)
-			(hide yes)
-			(show_name no)
-			(do_not_autoplace no)
-			(effects
-				(font
-					(size 1.27 1.27)
-				)
-			)
-		)
-		(property "Datasheet" ""
-			(at 81.28 247.65 0)
-			(hide yes)
-			(show_name no)
-			(do_not_autoplace no)
-			(effects
-				(font
-					(size 1.27 1.27)
-				)
-			)
-		)
-		(property "Description" ""
-			(at 81.28 247.65 0)
-			(hide yes)
-			(show_name no)
-			(do_not_autoplace no)
-			(effects
-				(font
-					(size 1.27 1.27)
-				)
-			)
-		)
-		(pin "1"
-		)
-		(pin "2"
-		)
-		(instances
-			(project "RocketLocator"
-				(path "/e63e39d7-6ac0-4ffd-8aa3-1841a4541b55"
-					(reference "C39")
-					(unit 1)
-				)

Commit message: Space J12 battery pins and drop J3
J3 ("Battery-") was a separate pad so the battery leads could be
soldered apart. Return current through it ran along the bottom edge
past the U19 magnetometer. Instead, J12 now uses a 1x06 outline with
pads at positions 1-3 and 6 only, so +BATT sits 7.6 mm from the nearest
GND pad and every battery return enters at the top edge.

- New footprint Custom:PinHeader_1x06_P2.54mm_Vertical_Pos4-5_Empty.
  Pad numbers and nets are unchanged (1 GND, 2 MSW, 3 GND, 4 +BATT).
  Pad 4 is moved to position 6.
- Remove J3 and its GND symbol from the schematic.
- BOM: J12 footprint updated, J3 row removed (table now A1:Q53).

The PCB is not updated in this commit; run Update PCB from Schematic.

Co-Authored-By: Claude Opus 5.5 (1M context) <noreply@anthropic.com>
Claude-Session: https://claude.ai/code/session_01FYY8Uv6gBjRSv3QTZNtnYK
Parts:
- removed J3: Battery-, Custom:PinHeader_1x01_P2.54mm_Vertical, symbol Connector:Conn_01x01_Female
- J12: footprint Custom:PinHeader_1x04_P2.54mm_Vertical -> Custom:PinHeader_1x06_P2.54mm_Vertical_Pos4-5_Empty
Changed lines of the file:
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@@
 	)
 	(symbol
-		(lib_id "Connector:Conn_01x01_Female")
-		(at 121.92 87.63 0)
-		(mirror x)
-		(unit 1)
-		(body_style 1)
-		(exclude_from_sim no)
-		(in_bom yes)
-		(on_board yes)
-		(in_pos_files yes)
-		(dnp no)
-		(property "Reference" "J3"
-			(at 124.46 85.09 0)
-			(show_name no)
-			(do_not_autoplace no)
-			(effects
-				(font
-					(size 1.27 1.27)
-				)
-			)
-		)
-		(property "Value" "Battery-"
-			(at 127 87.63 0)
-			(show_name no)
-			(do_not_autoplace no)
-			(effects
-				(font
-					(size 1.27 1.27)
-				)
-			)
-		)
-		(property "Footprint" "Custom:PinHeader_1x01_P2.54mm_Vertical"
-			(at 121.92 87.63 0)
-			(hide yes)
-			(show_name no)
-			(do_not_autoplace no)
-			(effects
-				(font
-					(size 1.27 1.27)
-				)
-			)
-		)
-		(property "Datasheet" ""
-			(at 121.92 87.63 0)
-			(hide yes)
-			(show_name no)
-			(do_not_autoplace no)
-			(effects
-				(font
-					(size 1.27 1.27)
-				)
-			)
-		)
-		(property "Description" ""
-			(at 121.92 87.63 0)
-			(hide yes)
-			(show_name no)
-			(do_not_autoplace no)
-			(effects
-				(font
-					(size 1.27 1.27)
-				)
-			)
-		)
-		(pin "1"
-		)
-		(instances
-			(project "RocketLocator"
-				(path "/e63e39d7-6ac0-4ffd-8aa3-1841a4541b55"
-					(reference "J3")
-					(unit 1)
-				)
-			)
-		)
-	)
-	(symbol
 		(lib_id "power:GND")
 		(at 19.05 199.39 0)
@@
 			)
 		)
-		(property "Footprint" "Custom:PinHeader_1x04_P2.54mm_Vertical"
+		(property "Footprint" "Custom:PinHeader_1x06_P2.54mm_Vertical_Pos4-5_Empty"
 			(at 121.92 72.39 0)
 			(hide yes)
@@
 					(unit 1)
 				)
-			)
-		)
-	)
-	(symbol
-		(lib_id "power:GND")
-		(at 116.84 87.63 0)
-		(mirror y)
-		(unit 1)
-		(body_style 1)
-		(exclude_from_sim no)
-		(in_bom yes)
-		(on_board yes)
-		(in_pos_files yes)
-		(dnp no)
-		(property "Reference" "#GND0149"
-			(at 116.84 93.98 0)
-			(hide yes)
-			(show_name no)
-			(do_not_autoplace no)
-			(effects
-				(font
-					(size 1.27 1.27)
-				)
-			)
-		)
-		(property "Value" "GND"
-			(at 116.713 92.0242 0)
-			(show_name no)
-			(do_not_autoplace no)
-			(effects
-				(font
-					(size 1.27 1.27)
-				)
-			)
-		)
-		(property "Footprint" ""
-			(at 116.84 87.63 0)
-			(hide yes)
-			(show_name no)
-			(do_not_autoplace no)
-			(effects
-				(font
-					(size 1.27 1.27)
-				)
-			)
-		)
-		(property "Datasheet" ""
-			(at 116.84 87.63 0)
-			(hide yes)
-			(show_name no)
-			(do_not_autoplace no)
-			(effects
-				(font
-					(size 1.27 1.27)
-				)
-			)
-		)
-		(property "Description" ""
-			(at 116.84 87.63 0)
-			(hide yes)
-			(show_name no)
-			(do_not_autoplace no)
-			(effects
-				(font
-					(size 1.27 1.27)
-				)
-			)
-		)
-		(pin "1"
-		)
-		(instances
-			(project "RocketLocator"
-				(path "/e63e39d7-6ac0-4ffd-8aa3-1841a4541b55"
-					(reference "#GND0149")
-					(unit 1)
-				)
